Commit message: week 2 - perception upload

File: tuto_package/urdf/tuto_half_home.urdf (robot description, URDF)
Before this commit: robot tuto, 6 links, 5 joints
Links:
- link depth_camera_link: geometry collision box size=0.05 0.05 0.05; visual box size=0.05 0.05 0.05
- link lidar_link: mass 0.1 -> 0.0125; geometry collision cylinder length=0.02 radius=0.025; visual cylinder length=0.02 radius=0.025
- link link_0: mass 1 -> 0.25; geometry collision box size=0.75 0.5 0.6; visual box size=0.75 0.5 0.6
- link link_1: mass 1 -> 0.125; geometry collision cylinder length=0.125 radius=0.15; visual cylinder length=0.125 radius=0.15
- link link_1_clone: mass 1 -> 0.125; geometry collision cylinder length=0.125 radius=0.15; visual cylinder length=0.125 radius=0.15
- link link_2: mass 1 -> 0.125; geometry collision sphere radius=0.1; visual sphere radius=0.1
Joints:
- joint depth_camera_joint: origin xyz=0.0 0.0 0.35 rpy=0 0 3.1416 -> xyz=-0.25 0.0 0.375 rpy=0 0 3.1416
- joint lidar_joint: origin xyz=0 0 0.274738 rpy=0 0 3.1416 -> xyz=-0.25 0 0.337369 rpy=0 0 3.1416
- joint link_0_JOINT_0: origin xyz=0.45 -0.625029 -0.1 rpy=1.5707 0 0 -> xyz=0.225 -0.3125145 -0.3 rpy=1.5707 0 0
- joint link_0_JOINT_1: origin xyz=0.45 0.625029 -0.1 rpy=1.5707 0 0 -> xyz=0.225 0.3125145 -0.3 rpy=1.5707 0 0
- joint link_0_JOINT_2: origin xyz=-0.55 0 -0.2 rpy=0 0 0 -> xyz=-0.275 0 -0.35 rpy=0 0 0

File: tuto_package/urdf/tuto_half_soccer.urdf (robot description, URDF)
Before this commit: robot tuto, 6 links, 5 joints
Links:
- link depth_camera_link: geometry collision box size=0.05 0.05 0.05; visual box size=0.05 0.05 0.05
- link lidar_link: mass 0.1 -> 0.0125; geometry collision cylinder length=0.02 radius=0.025; visual cylinder length=0.02 radius=0.025
- link link_0: mass 1 -> 0.125; geometry collision box size=0.75 0.5 0.2; visual box size=0.75 0.5 0.2
- link link_1: mass 1 -> 0.125; geometry collision cylinder length=0.125 radius=0.15; visual cylinder length=0.125 radius=0.15
- link link_1_clone: mass 1 -> 0.125; geometry collision cylinder length=0.125 radius=0.15; visual cylinder length=0.125 radius=0.15
- link link_2: mass 1 -> 0.125; geometry collision sphere radius=0.1; visual sphere radius=0.1
Joints:
- joint depth_camera_joint: origin xyz=0.0 0.0 0.35 rpy=0 0 3.1416 -> xyz=-0.25 0.0 0.175 rpy=0 0 3.1416
- joint lidar_joint: origin xyz=0 0 0.274738 rpy=0 0 3.1416 -> xyz=-0.25 0 0.137369 rpy=0 0 3.1416
- joint link_0_JOINT_0: origin xyz=0.45 -0.625029 -0.1 rpy=1.5707 0 0 -> xyz=0.225 -0.3125145 -0.05 rpy=1.5707 0 0
- joint link_0_JOINT_1: origin xyz=0.45 0.625029 -0.1 rpy=1.5707 0 0 -> xyz=0.225 0.3125145 -0.05 rpy=1.5707 0 0
- joint link_0_JOINT_2: origin xyz=-0.55 0 -0.2 rpy=0 0 0 -> xyz=-0.275 0 -0.1 rpy=0 0 0
